File: PCB/servo_pcb.kicad_sch (KiCad schematic)
At the start: 31 parts, among them M1 M1, M2 M2, M3 M2, M4 M2, M5 M2, U1 MM32G0001, U2 SL7533-3, U3 CP2119L, U4 INA180A2, U5 AS5600

Commit message: updated docs
Other:
- note added: "Motor Driver:CP2119L: 18v 5A"
- note removed: "Motor Driver:supports 2 drivers just need to use appropriate jumpers 1.BDR6121H : 7.5v 3A 2.CP2119L: 18v 5A"
Changed lines of the file:
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@@
 		)
 	)
-	(text "Motor Driver:supports 2 drivers\njust need to use appropriate jumpers\n1.BDR6121H : 7.5v 3A\n2.CP2119L: 18v 5A \n"
+	(text "Motor Driver:CP2119L: 18v 5A \n"
 		(exclude_from_sim no)
 		(at 57.15 73.406 0)

Commit message: docs: added OSHWA certification, contributing guide, and issue templates
Parts:
- R1: footprint Diode_SMD:D_2512_6332Metric_Pad1.52x3.35mm_HandSolder -> Resistor_SMD:R_2512_6332Metric_Pad1.40x3.35mm_HandSolder
Changed lines of the file:
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@@
 			)
 		)
-		(property "Footprint" "Diode_SMD:D_2512_6332Metric_Pad1.52x3.35mm_HandSolder"
+		(property "Footprint" "Resistor_SMD:R_2512_6332Metric_Pad1.40x3.35mm_HandSolder"
 			(at 141.478 40.64 90)
 			(effects
