File: PCB/servo_pcb_mg99x.kicad_sch (KiCad schematic)
At the start: 29 parts, among them J1 power in, M1 M1, M2 M2, U1 MM32G0001, U2 SL7533-3, U3 BDR6121H, U4 INA180A2, U5 AS5600

Commit message: docs: added OSHWA certification, contributing guide, and issue templates
Parts:
- R1: footprint Diode_SMD:D_2512_6332Metric_Pad1.52x3.35mm_HandSolder -> Resistor_SMD:R_2512_6332Metric_Pad1.40x3.35mm_HandSolder
Changed lines of the file:
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@@
 			)
 		)
-		(property "Footprint" "Diode_SMD:D_2512_6332Metric_Pad1.52x3.35mm_HandSolder"
+		(property "Footprint" "Resistor_SMD:R_2512_6332Metric_Pad1.40x3.35mm_HandSolder"
 			(at 141.478 40.64 90)
 			(effects
